Commit message: new branch

File: src/atvsim_description/models/ATV_agBOT/model.urdf (robot description, URDF)
Before this commit: robot ATV, 12 links, 11 joints
Links:
- removed link ATV/imu_link
- added link ATV_agBOT/imu_link, mass 0.015
- link base_link: geometry collision box size=0.01299 1.54 0.10226; collision box size=0.01299 1.54 0.10226
- link front_left_wheel: geometry collision cylinder length=0.2794 radius=0.3175; visual mesh filename=package://atvsim_description/models/ATV_agBOT/meshes/Wheel_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 scale=1.003700111 0.886200464 0.886200464
- link front_right_wheel: geometry collision cylinder length=0.2794 radius=0.3175; visual mesh filename=package://atvsim_description/models/ATV_agBOT/meshes/Wheel_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 scale=1.003700111 0.886200464 0.886200464
- link hokuyo_link: geometry collision box size=0.1 0.1 0.1; visual mesh filename=package://atvsim_description/models/ATV_agBOT/meshes/hokuyo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
- link rear_left_wheel: geometry collision cylinder length=0.2794 radius=0.3175; visual mesh filename=package://atvsim_description/models/ATV_agBOT/meshes/Wheels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 scale=1.003700111 0.886200464 0.886200464
- link rear_right_wheel: geometry collision cylinder length=0.2794 radius=0.3175; visual mesh filename=package://atvsim_description/models/ATV_agBOT/meshes/Wheels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 scale=1.003700111 0.886200464 0.886200464
Joints:
- removed joint ATV/imu_joint
- added joint ATV_agBOT/imu_joint: type fixed, parent base_link, child ATV_agBOT/imu_link, origin xyz=0  0  0 rpy=0  0  0, axis 1  0  0, limit lower=0.0 upper=0.0 effort=0.0 velocity=0.0
