Commit message: fixed ackermann, still need connect to ROS

File: src/atvsim_description/models/ATV/model.urdf (robot description, URDF)
Before this commit: robot ATV, 8 links, 7 joints
Links:
- added link steering_rod_left_block, mass 1; collision cylinder length=0.7 radius=0.01; visual cylinder length=1.22 radius=0.01
- added link steering_rod_right_block, mass 1; collision cylinder length=0.1 radius=0.01; visual cylinder length=0.1 radius=0.01
Joints:
- added joint front_left_steering_rod_joint: type continuous, parent front_left_wheel_steering_block, child steering_rod_left_block, origin xyz=0.5 0 -0.11 rpy=0  0       0, axis 0  1 0, limit lower=0 upper=0 effort=0.0 velocity=0.0
- added joint front_right_steering_rod_joint: type continuous, parent front_right_wheel_steering_block, child steering_rod_right_block, origin xyz=0.5 0 0.11 rpy=1.57079  0       0, axis 0  0  1, limit lower=0 upper=0 effort=0.0 velocity=0.0
- joint ATV/imu_joint: type revolute -> fixed

Commit message: driving with pub

File: src/atvsim_description/models/ATV/model.urdf (robot description, URDF)
Before this commit: robot ATV, 10 links, 9 joints
Joints:
- joint front_left_steering_rod_joint: origin xyz=0.5 0 -0.11 rpy=0  0       0 -> xyz=-0.5 0 0.11 rpy=0  0       0
- joint front_right_steering_rod_joint: origin xyz=0.5 0 0.11 rpy=1.57079  0       0 -> xyz=-0.5 0 -0.11 rpy=1.57079  0       0
- joint rear_left_wheel_joint: limit effort=0 velocity=0 -> effort=1000 velocity=5
- joint rear_right_wheel_joint: limit effort=0 velocity=0 -> effort=1000 velocity=5

Commit message: fully working with joystick, maybe tune pid a bit

File: src/atvsim_description/models/ATV/model.urdf (robot description, URDF)
Before this commit: robot ATV, 10 links, 9 joints
Links:
- link steering_rod_left_block: geometry collision cylinder length=0.7 radius=0.01; visual cylinder length=0.78 radius=0.01
Joints:
- joint front_right_steering_joint: limit lower=-0.7727 upper=0.7727 effort=0.0 velocity=0.0 -> lower=-0.7727 upper=0.7727 effort=1000 velocity=5
- joint rear_left_wheel_joint: limit effort=1000 velocity=5 -> effort=750 velocity=15
- joint rear_right_wheel_joint: limit effort=1000 velocity=5 -> effort=750 velocity=15

Commit message: bug in PPcontroller

File: src/atvsim_description/models/ATV/model.urdf (robot description, URDF)
Before this commit: robot ATV, 10 links, 9 joints
Joints:
- joint rear_left_wheel_joint: limit effort=750 velocity=15 -> effort=10000 velocity=1000
- joint rear_right_wheel_joint: limit effort=750 velocity=15 -> effort=10000 velocity=1000

Commit message: added camera & lidar simulation

File: src/atvsim_description/models/ATV/model.urdf (robot description, URDF)
Before this commit: robot ATV, 10 links, 9 joints
Links:
- removed link chassis
- added link base_link, mass 720.0; collision box size=0.01299 1.54 0.10226; collision box size=0.01299 1.54 0.10226
- added link camera_link, mass 1e-5; collision box size=0.05 0.05 0.05; visual box size=0.05 0.05 0.05
- added link hokuyo_link, mass 1e-5; collision box size=0.1 0.1 0.1; visual mesh filename=package://atvsim_description/models/ATV/meshes/hokuyo.dae
Joints:
- added joint camera_joint: type revolute, parent base_link, child camera_link, origin xyz=0.35 0 1.9 rpy=0 0 0, axis 0 1 0, limit lower=0 upper=0 effort=0.0 velocity=0.0
- added joint hokuyo_joint: type fixed, parent base_link, child hokuyo_link, origin xyz=1.2 0 1.1 rpy=0 0 0, axis 0 1 0
- joint ATV/imu_joint: parent chassis -> base_link
- joint front_left_steering_joint: parent chassis -> base_link
- joint front_right_steering_joint: parent chassis -> base_link
- joint rear_left_wheel_joint: parent chassis -> base_link
- joint rear_right_wheel_joint: parent chassis -> base_link

Commit message: tuned but not working yet

File: src/atvsim_description/models/ATV/model.urdf (robot description, URDF)
Before this commit: robot ATV, 12 links, 11 joints
Links:
- link base_link: mass 720.0 -> 1200.0

Commit message: latest config for hector

File: src/atvsim_description/models/ATV/model.urdf (robot description, URDF)
Before this commit: robot ATV, 12 links, 11 joints
Links:
- removed link ATV/imu_link
- added link imu_link, mass 0.015
Joints:
- removed joint ATV/imu_joint
- added joint imu_joint: type fixed, parent base_link, child imu_link, origin xyz=0  0  0 rpy=0  0  0, axis 1  0  0, limit lower=0.0 upper=0.0 effort=0.0 velocity=0.0

Commit message: update a bunch of files

File: src/atvsim_description/models/ATV/model.urdf (robot description, URDF)
Before this commit: robot ATV, 12 links, 11 joints
Joints:
- joint hokuyo_joint: origin xyz=1.2 0 1.1 rpy=0 0 0 -> xyz=1.2 0 1.8 rpy=0 0 0

Commit message: latest version

File: src/atvsim_description/models/ATV/model.urdf (robot description, URDF)
Before this commit: robot ATV, 12 links, 11 joints
Joints:
- joint hokuyo_joint: origin xyz=1.2 0 1.8 rpy=0 0 0 -> xyz=1.2 0 1.2 rpy=0 0 0

Commit message: git rid of backup

File: src/atvsim_description/models/ATV/model.urdf (robot description, URDF)
Before this commit: robot ATV, 12 links, 11 joints
Joints:
- joint hokuyo_joint: origin xyz=1.2 0 1.2 rpy=0 0 0 -> xyz=1.2 0 1.8 rpy=0 0 0
